Commit message: updated for real robot

File: src/vehicle_simulator/urdf/lidar.urdf.xacro (robot description, xacro)
@@ -3,6 +3,10 @@
   <link name="lidar" />
   <xacro:include filename="$(find velodyne_description)/urdf/VLP-16.urdf.xacro"/>
+  <xacro:include filename="$(find vehicle_simulator)/urdf/imu.xacro" />
   <xacro:VLP-16 parent="lidar" name="velodyne" topic="/velodyne_points" hz="6.3" samples="350" min_range="0.1">
     <origin xyz="0 0 0" rpy="0 0 0" />
   </xacro:VLP-16>
+  <xacro:imu parent_prefix="lidar" frame_prefix="imu">
+      <origin xyz="0.0 0 0.0" rpy="0 0 0"/>
+  </xacro:imu>
 </robot>
